Commit message: modification on my urdf of the robot

File: src/health_bot_description/urdf/inertials.xacro (robot description, xacro)
@@ -1,4 +1,4 @@
 <?xml version="1.0"?>
-<robot xmlns:xacro="http://www.ros.org">
+<robot  xmlns:xacro="http://www.ros.org/wiki/xacro">
     <!-- Macro for Sphere Inertia -->
     <xacro:macro name="inertial_sphere" params="mass radius *origin">

File: src/health_bot_description/urdf/robot.urdf.xacro (robot description, xacro)
@@ -1,4 +1,4 @@
 <?xml version="1.0"?>
-<robot name="health_bot" xmlns:xacro="http://www.ros.org">
+<robot name="health_bot" xmlns:xacro="http://www.ros.org/wiki/xacro">
     <xacro:include filename="inertials.xacro" />
     <material name="white"> <color rgba="1 1 1 1" /> </material>
@@ -64,25 +64,4 @@
         </xacro:inertial_sphere>
     </link>
-    <gazebo reference="chassis"> <material>Gazebo/Orange</material> </gazebo>
-    <gazebo reference="left_wheel"> <material>Gazebo/Blue</material> </gazebo>
-    <gazebo reference="right_wheel"> <material>Gazebo/Blue</material> </gazebo>
-    <gazebo reference="caster_wheel">
-        <material>Gazebo/Black</material>
-        <mu1 value="0.001" />
-        <mu2 value="0.001" />
-    </gazebo>
-    <gazebo>
-        <plugin filename="gz-sim-diff-drive-system" name="gz::sim::systems::DiffDrive">
-            <left_joint>left_wheel_joint</left_joint>
-            <right_joint>right_wheel_joint</right_joint>
-            <wheel_separation>0.35</wheel_separation>
-            <wheel_radius>0.1</wheel_radius>
-            <topic>cmd_vel</topic>
-            <odom_topic>odom</odom_topic>
-            <frame_id>odom</frame_id>
-            <child_frame_id>base_link</child_frame_id>
-        </plugin>
-        <plugin filename="gz-sim-joint-state-publisher-system" name="gz::sim::systems::JointStatePublisher"></plugin>
-    </gazebo>
     <!-- LiDAR JOINT -->
     <joint name="laser_joint" type="fixed">
@@ -108,4 +87,12 @@
         </xacro:inertial_cylinder>
     </link>
+     <gazebo reference="chassis"> <material>Gazebo/Orange</material> </gazebo>
+    <gazebo reference="left_wheel"> <material>Gazebo/Blue</material> </gazebo>
+    <gazebo reference="right_wheel"> <material>Gazebo/Blue</material> </gazebo>
+    <gazebo reference="caster_wheel">
+        <material>Gazebo/Black</material>
+        <mu1 value="0.001" />
+        <mu2 value="0.001" />
+    </gazebo>
     <gazebo reference="laser_frame">
         <material>Gazebo/Black</material>
@@ -131,3 +118,16 @@
         </sensor>
     </gazebo>
+    <gazebo>
+        <plugin filename="gz-sim-diff-drive-system" name="gz::sim::systems::DiffDrive">
+            <left_joint>left_wheel_joint</left_joint>
+            <right_joint>right_wheel_joint</right_joint>
+            <wheel_separation>0.35</wheel_separation>
+            <wheel_radius>0.1</wheel_radius>
+            <topic>cmd_vel</topic>
+            <odom_topic>odom</odom_topic>
+            <frame_id>odom</frame_id>
+            <child_frame_id>base_link</child_frame_id>
+        </plugin>
+        <plugin filename="gz-sim-joint-state-publisher-system" name="gz::sim::systems::JointStatePublisher"></plugin>
+    </gazebo>
 </robot>

Commit message: refactore my code in urdf

File: src/health_bot_description/urdf/inertials.xacro (robot description, xacro)
@@ -1,33 +1,69 @@
 <?xml version="1.0"?>
 <robot  xmlns:xacro="http://www.ros.org/wiki/xacro">
-    <!-- Macro for Sphere Inertia -->
-    <xacro:macro name="inertial_sphere" params="mass radius *origin">
+    <!-- #########################################-->
+    <!--             Mass and Inertia       -->
+    <!-- #########################################-->
+    <!-- here we assumed that all the links are made of the same material-->
+    <!-- body material density-->
+    <xacro:property name="d1" value="2710.0"/>
+    <!-- wheel material density-->
+    <xacro:property name="d2" value="2710.0"/>
+    <!-- caster wheel material density -->
+    <xacro:property name="d3" value="2710.0"/>
+    <!-- Robot body mass, wheel mass, center mass-->
+    <!--  body -->
+    <xacro:property name="m1" value="${d1 * a * b * c}"/>
+    <!-- wheel -->
+    <xacro:property name="m2" value="${d2 * pi * r * r * d}"/>
+    <!-- caster wheel -->
+    <xacro:property name="m3" value="${d3 * (4/3) * pi * r * r * r}"/>
+    <!-- moments of inertia of the robot body-->
+    <xacro:property name="Ix_body" value="${m1 * (b*b + c*c) / 12}" />
+    <xacro:property name="Iy_body" value="${m1 * (a*a + c*c) / 12}" />
+    <xacro:property name="Iz_body" value="${m1 * (a*a + b*b) / 12}" />
+    <!-- moments of inertia of the wheel -->
+    <xacro:property name="Iz_wheel" value="${0.5 * m2 * r * r}" />
+    <!-- here ix_wheel and iz_wheel is simillar-->
+    <xacro:property name="I_wheel" value="${(1.0/12.0) * m2 * (3.0*r*r + d*d)}" />
+     <!-- moment of inertais of the caster wheel sphere -->
+    <xacro:property name="I_caster" value="${(2.0/5.0) * m3 * r * r}" />
+    <!--###########################################-->
+    <!--    this macro defines the complete inertial section of the robot body-->
+    <!-- it is used later -->
+    <xacro:macro name="inertial_body">
         <inertial>
-            <xacro:insert_block name="origin"/>
-            <mass value="${mass}" />
-            <inertia ixx="${(2/5) * mass * (radius*radius)}" ixy="0.0" ixz="0.0"
-                     iyy="${(2/5) * mass * (radius*radius)}" iyz="0.0"
-                     izz="${(2/5) * mass * (radius*radius)}" />
+        <!-- displacement and the orientation of the center of the mass frames of the link with respect to the -->
+            <origin rpy="0 0 0" xyz="0 0 ${s1}"/>
+            <mass value="${m1}" />
+            <inertia ixx="${Ix_body}" ixy="0.0" ixz="0.0"
+                     iyy="${Iy_body}" iyz="0.0"
+                     izz="${Iz_body}" />
         </inertial>
     </xacro:macro>
-    <!-- Macro for Box Inertia -->
-    <xacro:macro name="inertial_box" params="mass x y z *origin">
-        <inertial>
-            <xacro:insert_block name="origin"/>
-            <mass value="${mass}" />
-            <inertia ixx="${(1/12) * mass * (y*y+z*z)}" ixy="0.0" ixz="0.0"
-                     iyy="${(1/12) * mass * (x*x+z*z)}" iyz="0.0"
-                     izz="${(1/12) * mass * (x*x+y*y)}" />
-        </inertial>
-    </xacro:macro>
-    <!-- Macro for Cylinder Inertia -->
-    <xacro:macro name="inertial_cylinder" params="mass length radius *origin">
-        <inertial>
-            <xacro:insert_block name="origin"/>
-            <mass value="${mass}" />
-            <inertia ixx="${(1/12) * mass * (3*radius*radius + length*length)}" ixy="0.0" ixz="0.0"
-                     iyy="${(1/12) * mass * (3*radius*radius + length*length)}" iyz="0.0"
-                     izz="${(1/2) * mass * (radius*radius)}" />
-        </inertial>
-    </xacro:macro>
+<!--###########################################-->
+<!--    this macro defines the complete inertial section of the wheel-->
+<!-- it is used later -->
+<xacro:macro name="inertial_wheel" >
+    <inertial>
+        <!-- displacement and the orientation of the center of the mass frames of the link with respect to the -->
+        <origin rpy="1.570795 0 0" xyz="0 0 0"/>
+        <mass value="${m2}" />
+        <inertia ixx="${I_wheel}" ixy="0.0" ixz="0.0"
+                 iyy="${I_wheel}" iyz="0.0"
+                 izz="${Iz_wheel}" />
+    </inertial>
+</xacro:macro>
+<!--###########################################-->
+<!--    this macro defines the complete inertial section of the caster wheel-->
+<!-- it is used later -->
+<xacro:macro name="inertial_caster" >
+    <inertial>
+        <!-- displacement and the orientation of the center of the mass frames of the link with respect to the -->
+        <origin rpy="0 0 0" xyz="0 0 0"/>
+        <mass value="${m3}" />
+        <inertia ixx="${I_caster}" ixy="0.0" ixz="0.0"
+                 iyy="${I_caster}" iyz="0.0"
+                 izz="${I_caster}" />
+    </inertial>
+</xacro:macro>
 </robot>

File: src/health_bot_description/urdf/robot.urdf.xacro (robot description, xacro)
@@ -1,133 +1,119 @@
 <?xml version="1.0"?>
 <robot name="health_bot" xmlns:xacro="http://www.ros.org/wiki/xacro">
+    <!-- include the inertial-->
     <xacro:include filename="inertials.xacro" />
-    <material name="white"> <color rgba="1 1 1 1" /> </material>
-    <material name="blue"> <color rgba="0.2 0.2 1 1" /> </material>
-    <material name="black"> <color rgba="0 0 0 1" /> </material>
-    <link name="base_link"></link>
-    <joint name="chassis_joint" type="fixed">
-        <parent link="base_link" />
-        <child link="chassis" />
-        <origin xyz="-0.1 0 0" />
-    </joint>
-    <link name="chassis">
-        <visual>
-            <origin xyz="0.25 0 0.075" />
-            <geometry> <box size="0.5 0.3 0.15" /> </geometry>
-            <material name="white" />
-        </visual>
-        <collision>
-            <origin xyz="0.25 0 0.075" />
-            <geometry> <box size="0.5 0.3 0.15" /> </geometry>
-        </collision>
-        <xacro:inertial_box mass="0.5" x="0.5" y="0.3" z="0.15">
-            <origin xyz="0.25 0 0.075" rpy="0 0 0" />
-        </xacro:inertial_box>
-    </link>
-    <xacro:macro name="wheel" params="prefix y_reflect">
-        <joint name="${prefix}_wheel_joint" type="continuous">
-            <parent link="base_link" />
-            <child link="${prefix}_wheel" />
-            <origin xyz="0 ${y_reflect * 0.175} 0" rpy="-${pi/2} 0 0" />
-            <axis xyz="0 0 1" />
-        </joint>
-        <link name="${prefix}_wheel">
-            <visual>
-                <geometry> <cylinder radius="0.1" length="0.04" /> </geometry>
-                <material name="blue" />
-            </visual>
-            <collision>
-                <geometry> <cylinder radius="0.1" length="0.04" /> </geometry>
-            </collision>
-            <xacro:inertial_cylinder mass="0.1" length="0.04" radius="0.1">
-                <origin xyz="0 0 0" rpy="0 0 0" />
-            </xacro:inertial_cylinder>
-        </link>
-    </xacro:macro>
-    <xacro:wheel prefix="left" y_reflect="1" />
-    <xacro:wheel prefix="right" y_reflect="-1" />
-    <joint name="caster_wheel_joint" type="fixed">
-        <parent link="chassis" />
-        <child link="caster_wheel" />
-        <origin xyz="0.4 0 0" />
-    </joint>
-    <link name="caster_wheel">
-        <visual>
-            <geometry> <sphere radius="0.05" /> </geometry>
-            <material name="black" />
-        </visual>
-        <collision>
-            <geometry> <sphere radius="0.05" /> </geometry>
-        </collision>
-        <xacro:inertial_sphere mass="0.1" radius="0.05">
-            <origin xyz="0 0 0" rpy="0 0 0" />
-        </xacro:inertial_sphere>
-    </link>
-    <!-- LiDAR JOINT -->
-    <joint name="laser_joint" type="fixed">
-        <parent link="chassis"/>
-        <child link="laser_frame"/>
-        <origin xyz="0.1 0 0.175" rpy="0 0 0"/>
-    </joint>
-    <!-- LiDAR LINK -->
-    <link name="laser_frame">
-        <visual>
-            <geometry>
-                <cylinder radius="0.05" length="0.04"/>
-            </geometry>
-            <material name="black"/>
-        </visual>
-        <collision>
-            <geometry>
-                <cylinder radius="0.05" length="0.04"/>
-            </geometry>
-        </collision>
-        <xacro:inertial_cylinder mass="0.1" length="0.04" radius="0.05">
-            <origin xyz="0 0 0" rpy="0 0 0"/>
-        </xacro:inertial_cylinder>
-    </link>
-     <gazebo reference="chassis"> <material>Gazebo/Orange</material> </gazebo>
-    <gazebo reference="left_wheel"> <material>Gazebo/Blue</material> </gazebo>
-    <gazebo reference="right_wheel"> <material>Gazebo/Blue</material> </gazebo>
-    <gazebo reference="caster_wheel">
-        <material>Gazebo/Black</material>
-        <mu1 value="0.001" />
-        <mu2 value="0.001" />
-    </gazebo>
-    <gazebo reference="laser_frame">
-        <material>Gazebo/Black</material>
-        <sensor name="laser" type="gpu_lidar">
-            <pose> 0 0 0 0 0 0 </pose>
-            <visualize>true</visualize>
-            <update_rate>10</update_rate>
-            <lidar>
-                <scan>
-                    <horizontal>
-                        <samples>360</samples>
-                        <min_angle>-3.14</min_angle>
-                        <max_angle>3.14</max_angle>
-                    </horizontal>
-                </scan>
-                <range>
-                    <min>0.3</min>
-                    <max>12</max>
-                </range>
-            </lidar>
-            <topic>scan</topic>
-            <!-- <gz_frame_id>laser_frame</gz_frame_id> -->
-        </sensor>
-    </gazebo>
-    <gazebo>
-        <plugin filename="gz-sim-diff-drive-system" name="gz::sim::systems::DiffDrive">
-            <left_joint>left_wheel_joint</left_joint>
-            <right_joint>right_wheel_joint</right_joint>
-            <wheel_separation>0.35</wheel_separation>
-            <wheel_radius>0.1</wheel_radius>
-            <topic>cmd_vel</topic>
-            <odom_topic>odom</odom_topic>
-            <frame_id>odom</frame_id>
-            <child_frame_id>base_link</child_frame_id>
-        </plugin>
-        <plugin filename="gz-sim-joint-state-publisher-system" name="gz::sim::systems::JointStatePublisher"></plugin>
-    </gazebo>
+    <!-- Define the pi constants -->
+    <xacro:property name="pi" value="3.14159265359" />
+    <!-- define the body dimension-->
+    <xacro:property name="a" value="1" />
+    <xacro:property name="b" value="0.3" />
+    <xacro:property name="c" value="0.6" />
+    <!-- define the wheel and the caster dimensions-->
+    <!-- define the wheel and the caster radius-->
+    <xacro:property name="r" value="0.15"/>
+    <!-- define the wheel width-->
+    <xacro:property name="d" value="0.1"/>
+    <xacro:property name="s1" value="${b/2+r}"/>
+    <xacro:property name="s2" value="${2 * r}"/>
+    <xacro:property name="s3" value="${2*r}"/>
+    <xacro:property name="s4" value="${c/2+d/2}"/>
+<!--##################################################-->
+<!--   here additional file will be needed for the robot gazebo we will come back here-->
+<!--  we need this link otherwise gazebo will complain-->
+ <xacro:include filename="robot.gazebo" />
+<link name="base_footprint"></link>
+<joint name="base_footprint_joint" type="fixed">
+    <parent link="base_footprint" />
+    <child link="body_link" />
+</joint>
+<!-- the above is just the fictious link fo the robot -->
+<!-- below is the body link of the robot-->
+<link name="body_link">
+    <visual>
+<origin rpy="0 0 0" xyz="0 0 ${s1}"/>
+    <geometry>
+        <box size="${a} ${b} ${c}" />
+    </geometry>
+    <!-- here the displacement an dthe orientation of the geometric center of the link with respect to the link-->
+</visual>
+<collision>
+<origin rpy="0 0 0" xyz="0 0 ${s1}"/>
+    <geometry>
+        <box size="${a} ${b} ${c}" />
+    </geometry>
+    <!-- here the displacement an dthe orientation of the geometric center of the link with respect to the link-->
+</collision>
+<xacro:inertial_body />
+</link>
+<!-- the next step is for the  back right wheel of the robot and the joint-->
+<joint name="wheel1_joint" type="continuous">
+    <parent link="body_link" />
+    <child link="wheel1_link" />
+    <origin xyz="${-s2} ${-s4} ${r}" rpy="0 0 0" />
+    <axis xyz="0 1 0" />
+    <limit effort="50000" velocity="10" />
+    <dynamics damping="1.0" friction="1.0" />
+</joint>
+<link name="wheel1_link">
+    <visual>
+       <origin rpy="1.570795 0 0" xyz="0 0 0"/>
+        <geometry>
+            <cylinder radius="${r}" length="${d}" />
+        </geometry>
+        <!-- here the displacement an dthe orientation of the geometric center of the link with respect to the link-->
+    </visual>
+    <collision>
+        <origin rpy="1.570795 0 0" xyz="0 0 0"/>
+        <geometry>
+            <cylinder radius="${r}" length="${d}" />
+        </geometry>
+        <!-- here the displacement an dthe orientation of the geometric center of the link with respect to the link-->
+    </collision>
+    <xacro:inertial_wheel />
+</link>
+<!-- the left wheel is the next one -->
+<joint name="wheel2_joint" type="continuous">
+    <parent link="body_link" />
+    <child link="wheel2_link" />
+    <origin xyz="${-s2} ${s4} ${r}" rpy="0 0 0" />
+    <axis xyz="0 1 0" />
+    <limit effort="50000" velocity="10" />
+    <dynamics damping="1.0" friction="1.0" />
+</joint>
+<link name="wheel2_link">
+    <visual>
+        <origin rpy="1.570795 0 0" xyz="0 0 0"/>
+        <geometry>
+            <cylinder radius="${r}" length="${d}" />
+        </geometry>
+    </visual>
+    <collision>
+        <origin rpy="1.570795 0 0" xyz="0 0 0"/>
+        <geometry>
+            <cylinder radius="${r}" length="${d}" />
+        </geometry>
+    </collision>
+    <xacro:inertial_wheel />
+</link>
+<!-- for the caster wheel -->
+<joint name="caster_joint" type="fixed">
+    <parent link="body_link" />
+    <child link="caster_link" />
+    <origin xyz="${s3} 0 ${r}" rpy="0 0 0" />
+</joint>
+<link name="caster_link">
+    <visual>
+        <origin rpy="0 0 0" xyz="0 0 0"/>
+        <geometry>
+            <sphere radius="${r}" />
+        </geometry>
+    </visual>
+    <collision>
+        <origin rpy="0 0 0" xyz="0 0 0"/>
+        <geometry>
+            <sphere radius="${r}" />
+        </geometry>
+    </collision>
+    <xacro:inertial_caster />
+</link>
 </robot>
