Commit message: refactor the structure of my code

File: src/health_bot_description/urdf/inertials.xacro (robot description, xacro)
@@ -1,38 +1,26 @@
 <?xml version="1.0"?>
-<robot  xmlns:xacro="http://www.ros.org/wiki/xacro">
-    <!-- #########################################-->
-    <!--             Mass and Inertia       -->
-    <!-- #########################################-->
-    <!-- here we assumed that all the links are made of the same material-->
-    <!-- body material density-->
-    <xacro:property name="d1" value="2710.0"/>
-    <!-- wheel material density-->
-    <xacro:property name="d2" value="2710.0"/>
-    <!-- caster wheel material density -->
-    <xacro:property name="d3" value="2710.0"/>
-    <!-- Robot body mass, wheel mass, center mass-->
-    <!--  body -->
+<robot xmlns:xacro="http://www.ros.org/wiki/xacro">
+    <!-- Material Densities (kg/m^3) - 600 is stable for simulation -->
+    <xacro:property name="d1" value="600.0"/>
+    <xacro:property name="d2" value="600.0"/>
+    <xacro:property name="d3" value="600.0"/>
+    <!-- Mass Calculations -->
     <xacro:property name="m1" value="${d1 * a * b * c}"/>
-    <!-- wheel -->
     <xacro:property name="m2" value="${d2 * pi * r * r * d}"/>
-    <!-- caster wheel -->
-    <xacro:property name="m3" value="${d3 * (4/3) * pi * r * r * r}"/>
-    <!-- moments of inertia of the robot body-->
+    <xacro:property name="m3" value="${d3 * (4/3) * pi * cr * cr * cr}"/>
+    <!-- Body Inertia Moments (Box) -->
     <xacro:property name="Ix_body" value="${m1 * (b*b + c*c) / 12}" />
     <xacro:property name="Iy_body" value="${m1 * (a*a + c*c) / 12}" />
     <xacro:property name="Iz_body" value="${m1 * (a*a + b*b) / 12}" />
-    <!-- moments of inertia of the wheel -->
+    <!-- Wheel Inertia Moments (Cylinder) -->
+    <!-- When cylinder is rotated pi/2 on X, Iz becomes the rolling axis -->
     <xacro:property name="Iz_wheel" value="${0.5 * m2 * r * r}" />
-    <!-- here ix_wheel and iz_wheel is simillar-->
     <xacro:property name="I_wheel" value="${(1.0/12.0) * m2 * (3.0*r*r + d*d)}" />
-     <!-- moment of inertais of the caster wheel sphere -->
-    <xacro:property name="I_caster" value="${(2.0/5.0) * m3 * r * r}" />
-    <!--###########################################-->
-    <!--    this macro defines the complete inertial section of the robot body-->
-    <!-- it is used later -->
+    <!-- Caster Inertia Moments (Sphere) -->
+    <xacro:property name="I_caster" value="${(2.0/5.0) * m3 * cr * cr}" />
+    <!-- BODY INERTIA MACRO -->
     <xacro:macro name="inertial_body">
         <inertial>
-        <!-- displacement and the orientation of the center of the mass frames of the link with respect to the -->
-            <origin rpy="0 0 0" xyz="0 0 ${s1}"/>
+            <origin rpy="0 0 0" xyz="0 0 ${c/2}" />
             <mass value="${m1}" />
             <inertia ixx="${Ix_body}" ixy="0.0" ixz="0.0"
@@ -41,29 +29,24 @@
         </inertial>
     </xacro:macro>
-<!--###########################################-->
-<!--    this macro defines the complete inertial section of the wheel-->
-<!-- it is used later -->
-<xacro:macro name="inertial_wheel" >
-    <inertial>
-        <!-- displacement and the orientation of the center of the mass frames of the link with respect to the -->
-        <origin rpy="1.570795 0 0" xyz="0 0 0"/>
-        <mass value="${m2}" />
-        <inertia ixx="${I_wheel}" ixy="0.0" ixz="0.0"
-                 iyy="${I_wheel}" iyz="0.0"
-                 izz="${Iz_wheel}" />
-    </inertial>
-</xacro:macro>
-<!--###########################################-->
-<!--    this macro defines the complete inertial section of the caster wheel-->
-<!-- it is used later -->
-<xacro:macro name="inertial_caster" >
-    <inertial>
-        <!-- displacement and the orientation of the center of the mass frames of the link with respect to the -->
-        <origin rpy="0 0 0" xyz="0 0 0"/>
-        <mass value="${m3}" />
-        <inertia ixx="${I_caster}" ixy="0.0" ixz="0.0"
-                 iyy="${I_caster}" iyz="0.0"
-                 izz="${I_caster}" />
-    </inertial>
-</xacro:macro>
+    <!-- WHEEL INERTIA MACRO -->
+    <xacro:macro name="inertial_wheel">
+        <inertial>
+            <!-- Important: Orientation of mass must match visual orientation -->
+            <origin rpy="${pi/2} 0 0" xyz="0 0 0"/>
+            <mass value="${m2}" />
+            <inertia ixx="${I_wheel}" ixy="0.0" ixz="0.0"
+                     iyy="${I_wheel}" iyz="0.0"
+                     izz="${Iz_wheel}" />
+        </inertial>
+    </xacro:macro>
+    <!-- CASTER INERTIA MACRO -->
+    <xacro:macro name="inertial_caster">
+        <inertial>
+            <origin rpy="0 0 0" xyz="0 0 0"/>
+            <mass value="${m3}" />
+            <inertia ixx="${I_caster}" ixy="0.0" ixz="0.0"
+                     iyy="${I_caster}" iyz="0.0"
+                     izz="${I_caster}" />
+        </inertial>
+    </xacro:macro>
 </robot>

File: src/health_bot_description/urdf/robot.urdf.xacro (robot description, xacro)
@@ -1,119 +1,73 @@
 <?xml version="1.0"?>
 <robot name="health_bot" xmlns:xacro="http://www.ros.org/wiki/xacro">
-    <!-- include the inertial-->
+    <!-- 1. PHYSICAL DIMENSIONS (Defined First) -->
+    <xacro:property name="a" value="0.6" /> <!-- Length (X) -->
+    <xacro:property name="b" value="0.4" /> <!-- Width (Y) -->
+    <xacro:property name="c" value="0.3" /> <!-- Height (Z) -->
+    <!-- WHEEL DIMENSIONS -->
+    <xacro:property name="r" value="0.1" />  <!-- Drive Wheel Radius -->
+    <xacro:property name="d" value="0.05" /> <!-- Drive Wheel Width -->
+    <xacro:property name="cr" value="0.1" /> <!-- Caster Radius -->
+    <!-- 2. CALCULATED OFFSETS (Defined Second) -->
+    <!-- <xacro:property name="chassis_z_offset" value="${(c/2) + r}" /> -->
+    <xacro:property name="wheel_y_offset" value="${(b/2) + (d/2)}" />
+    <!-- <xacro:property name="wheel_x_offset" value="0.15" /> -->
+    <!-- 3. INCLUDE EXTERNAL FILES (Now they can see the variables above) -->
     <xacro:include filename="inertials.xacro" />
-    <!-- Define the pi constants -->
-    <xacro:property name="pi" value="3.14159265359" />
-    <!-- define the body dimension-->
-    <xacro:property name="a" value="1" />
-    <xacro:property name="b" value="0.3" />
-    <xacro:property name="c" value="0.6" />
-    <!-- define the wheel and the caster dimensions-->
-    <!-- define the wheel and the caster radius-->
-    <xacro:property name="r" value="0.15"/>
-    <!-- define the wheel width-->
-    <xacro:property name="d" value="0.1"/>
-    <xacro:property name="s1" value="${b/2+r}"/>
-    <xacro:property name="s2" value="${2 * r}"/>
-    <xacro:property name="s3" value="${2*r}"/>
-    <xacro:property name="s4" value="${c/2+d/2}"/>
-<!--##################################################-->
-<!--   here additional file will be needed for the robot gazebo we will come back here-->
-<!--  we need this link otherwise gazebo will complain-->
- <xacro:include filename="robot.gazebo" />
-<link name="base_footprint"></link>
-<joint name="base_footprint_joint" type="fixed">
-    <parent link="base_footprint" />
-    <child link="body_link" />
-</joint>
-<!-- the above is just the fictious link fo the robot -->
-<!-- below is the body link of the robot-->
-<link name="body_link">
-    <visual>
-<origin rpy="0 0 0" xyz="0 0 ${s1}"/>
-    <geometry>
-        <box size="${a} ${b} ${c}" />
-    </geometry>
-    <!-- here the displacement an dthe orientation of the geometric center of the link with respect to the link-->
-</visual>
-<collision>
-<origin rpy="0 0 0" xyz="0 0 ${s1}"/>
-    <geometry>
-        <box size="${a} ${b} ${c}" />
-    </geometry>
-    <!-- here the displacement an dthe orientation of the geometric center of the link with respect to the link-->
-</collision>
-<xacro:inertial_body />
-</link>
-<!-- the next step is for the  back right wheel of the robot and the joint-->
-<joint name="wheel1_joint" type="continuous">
-    <parent link="body_link" />
-    <child link="wheel1_link" />
-    <origin xyz="${-s2} ${-s4} ${r}" rpy="0 0 0" />
-    <axis xyz="0 1 0" />
-    <limit effort="50000" velocity="10" />
-    <dynamics damping="1.0" friction="1.0" />
-</joint>
-<link name="wheel1_link">
-    <visual>
-       <origin rpy="1.570795 0 0" xyz="0 0 0"/>
-        <geometry>
-            <cylinder radius="${r}" length="${d}" />
-        </geometry>
-        <!-- here the displacement an dthe orientation of the geometric center of the link with respect to the link-->
-    </visual>
-    <collision>
-        <origin rpy="1.570795 0 0" xyz="0 0 0"/>
-        <geometry>
-            <cylinder radius="${r}" length="${d}" />
-        </geometry>
-        <!-- here the displacement an dthe orientation of the geometric center of the link with respect to the link-->
-    </collision>
-    <xacro:inertial_wheel />
-</link>
-<!-- the left wheel is the next one -->
-<joint name="wheel2_joint" type="continuous">
-    <parent link="body_link" />
-    <child link="wheel2_link" />
-    <origin xyz="${-s2} ${s4} ${r}" rpy="0 0 0" />
-    <axis xyz="0 1 0" />
-    <limit effort="50000" velocity="10" />
-    <dynamics damping="1.0" friction="1.0" />
-</joint>
-<link name="wheel2_link">
-    <visual>
-        <origin rpy="1.570795 0 0" xyz="0 0 0"/>
-        <geometry>
-            <cylinder radius="${r}" length="${d}" />
-        </geometry>
-    </visual>
-    <collision>
-        <origin rpy="1.570795 0 0" xyz="0 0 0"/>
-        <geometry>
-            <cylinder radius="${r}" length="${d}" />
-        </geometry>
-    </collision>
-    <xacro:inertial_wheel />
-</link>
-<!-- for the caster wheel -->
-<joint name="caster_joint" type="fixed">
-    <parent link="body_link" />
-    <child link="caster_link" />
-    <origin xyz="${s3} 0 ${r}" rpy="0 0 0" />
-</joint>
-<link name="caster_link">
-    <visual>
-        <origin rpy="0 0 0" xyz="0 0 0"/>
-        <geometry>
-            <sphere radius="${r}" />
-        </geometry>
-    </visual>
-    <collision>
-        <origin rpy="0 0 0" xyz="0 0 0"/>
-        <geometry>
-            <sphere radius="${r}" />
-        </geometry>
-    </collision>
-    <xacro:inertial_caster />
-</link>
+    <xacro:include filename="robot.gazebo" />
+    <!-- 4. ROBOT STRUCTURE -->
+    <link name="base_footprint"></link>
+    <joint name="base_joint" type="fixed">
+        <parent link="base_footprint" />
+        <child link="body_link" />
+        <origin xyz="0 0 ${r}" rpy="0 0 0" />
+    </joint>
+    <link name="body_link">
+        <visual>
+            <origin xyz="0 0 ${c/2}" rpy="0 0 0" />
+            <geometry> <box size="${a} ${b} ${c}" /> </geometry>
+        </visual>
+        <collision>
+            <origin xyz="0 0 ${c/2}" rpy="0 0 0" />
+            <geometry> <box size="${a} ${b} ${c}" /> </geometry>
+        </collision>
+        <xacro:inertial_body />
+    </link>
+    <!-- WHEEL MACRO -->
+    <xacro:macro name="m_wheel" params="prefix y_reflect">
+        <joint name="${prefix}_wheel_joint" type="continuous">
+            <parent link="body_link" />
+            <child link="${prefix}_wheel_link" />
+            <origin xyz="-0.15 ${y_reflect * wheel_y_offset} 0" rpy="0 0 0" />
+            <axis xyz="0 1 0" />
+        </joint>
+        <link name="${prefix}_wheel_link">
+            <visual>
+                <origin rpy="${pi/2} 0 0" xyz="0 0 0" />
+                <geometry> <cylinder radius="${r}" length="${d}" /> </geometry>
+            </visual>
+            <collision>
+                <origin rpy="${pi/2} 0 0" xyz="0 0 0" />
+                <geometry> <cylinder radius="${r}" length="${d}" /> </geometry>
+            </collision>
+            <xacro:inertial_wheel />
+        </link>
+    </xacro:macro>
+    <xacro:m_wheel prefix="right" y_reflect="-1" />
+    <xacro:m_wheel prefix="left" y_reflect="1" />
+    <!-- CASTER WHEEL (FRONT) -->
+    <joint name="caster_joint" type="fixed">
+        <parent link="body_link" />
+        <child link="caster_link" />
+        <origin xyz="0.2 0 0" rpy="0 0 0" />
+    </joint>
+    <link name="caster_link">
+        <visual>
+            <geometry> <sphere radius="${cr}" /> </geometry>
+        </visual>
+        <collision>
+            <geometry> <sphere radius="${cr}" /> </geometry>
+        </collision>
+        <xacro:inertial_caster />
+    </link>
 </robot>

Commit message: lidar sensor add

File: src/health_bot_description/urdf/inertials.xacro (robot description, xacro)
@@ -19,4 +19,8 @@
     <!-- Caster Inertia Moments (Sphere) -->
     <xacro:property name="I_caster" value="${(2.0/5.0) * m3 * cr * cr}" />
+    <!--lidar specification -->
+<xacro:property name="I_lidar_x" value="${(1/12) * laser_m * (3*laser_r*laser_r + laser_l*laser_l)}"/>
+<xacro:property name="I_lidar_y" value="${(1/12) * laser_m * (3*laser_r*laser_r + laser_l*laser_l)}"/>
+<xacro:property name="I_lidar_z" value="${(1/2) * laser_m * (laser_r*laser_r)}"/>
     <!-- BODY INERTIA MACRO -->
     <xacro:macro name="inertial_body">
@@ -50,3 +54,17 @@
         </inertial>
     </xacro:macro>
+   <!-- LIDAR INERTIA MACRO -->
+    <!-- Macro for LiDAR/Cylinder Inertia -->
+    <!-- LIDAR INERTIA MACRO -->
+<xacro:macro name="inertial_lidar">
+  <inertial>
+    <origin xyz="0 0 ${laser_l/2}" rpy="0 0 0"/>
+    <!-- Mass of the LiDAR sensor -->
+    <mass value="${laser_m}"/>
+    <!-- Approximate inertia values for a small cylindrical sensor -->
+    <inertia ixx="${I_lidar_x}" ixy="0.0" ixz="0.0"
+             iyy="${I_lidar_y}" iyz="0.0"
+             izz="${I_lidar_z}"/>
+  </inertial>
+</xacro:macro>
 </robot>

File: src/health_bot_description/urdf/robot.urdf.xacro (robot description, xacro)
@@ -1,4 +1,7 @@
 <?xml version="1.0"?>
 <robot name="health_bot" xmlns:xacro="http://www.ros.org/wiki/xacro">
+<material name="black">
+  <color rgba="0 0 0 1"/>
+</material>
     <!-- 1. PHYSICAL DIMENSIONS (Defined First) -->
     <xacro:property name="a" value="0.6" /> <!-- Length (X) -->
@@ -9,4 +12,8 @@
     <xacro:property name="d" value="0.05" /> <!-- Drive Wheel Width -->
     <xacro:property name="cr" value="0.1" /> <!-- Caster Radius -->
+       <!-- LiDAR PROPERTIES -->
+    <xacro:property name="laser_r" value="0.05" />
+    <xacro:property name="laser_l" value="0.04" />
+    <xacro:property name="laser_m" value="0.1" />
     <!-- 2. CALCULATED OFFSETS (Defined Second) -->
     <!-- <xacro:property name="chassis_z_offset" value="${(c/2) + r}" /> -->
@@ -71,3 +78,21 @@
         <xacro:inertial_caster />
     </link>
+    <!-- LiDAR JOINT (Top Front) -->
+    <joint name="laser_joint" type="fixed">
+        <parent link="body_link" />
+        <child link="laser_frame" />
+        <!-- Moves it to the front (+X) and on top of the chassis (+Z) -->
+         <origin xyz="0.2 0 ${c}" rpy="0 0 0" />
+    </joint>
+    <link name="laser_frame">
+        <visual>
+            <geometry> <cylinder radius="${laser_r}" length="${laser_l}" /> </geometry>
+            <material name="black" />
+        </visual>
+        <collision>
+            <geometry> <cylinder radius="${laser_r}" length="${laser_l}" /> </geometry>
+        </collision>
+        <!-- Using the NEW dynamic macro from inertials.xacro -->
+        <xacro:inertial_lidar/>
+    </link>
 </robot>
