Commit message: configuring custom SLAM toolbox for localization and mapping

File: src/health_bot_description/urdf/robot.urdf.xacro (robot description, xacro)
@@ -81,9 +81,9 @@
     <joint name="laser_joint" type="fixed">
         <parent link="body_link" />
-        <child link="laser_frame" />
-        <!-- Moves it to the front (+X) and on top of the chassis (+Z) -->
-         <origin xyz="0.2 0 ${c}" rpy="0 0 0" />
+        <child link="laser_link" />
+        <!--  -->
+         <origin xyz="0.2 0 ${c + laser_l/2}" rpy="0 0 0" />
     </joint>
-    <link name="laser_frame">
+    <link name="laser_link">
         <visual>
             <geometry> <cylinder radius="${laser_r}" length="${laser_l}" /> </geometry>
@@ -93,5 +93,4 @@
             <geometry> <cylinder radius="${laser_r}" length="${laser_l}" /> </geometry>
         </collision>
-        <!-- Using the NEW dynamic macro from inertials.xacro -->
         <xacro:inertial_lidar/>
     </link>
