Commit message: bug fixed

File: src/health_bot_description/urdf/healthbot.urdf.xacro (robot description, xacro)
@@ -7,6 +7,7 @@
   <!-- Include Gazebo Parameters -->
   <xacro:include filename="$(find health_bot_description)/urdf/healthbot_gazebo.xacro" />
-  <!-- Include ros2_control Plugins
-  <xacro:include filename="$(find health_bot_description)/urdf/health_bot_ros2_control.xacro" /> -->
+<!--
+  Include ros2_control Plugins -->
+  <!-- <xacro:include filename="$(find health_bot_description)/urdf/healthbot_ros2_control.xacro" /> -->
   <link name="base_footprint"/>
   <link name="base_link">

File: src/health_bot_description/urdf/healthbot_gazebo.xacro (robot description, xacro)
@@ -41,8 +41,8 @@
   <!-- ROS 2 Control + Sensors (Gazebo Harmonic) -->
   <gazebo>
-  <plugin filename="gz_ros2_control-system"
+  <!-- <plugin filename="gz_ros2_control-system"
    name="gz_ros2_control::GazeboSimROS2ControlPlugin">
    <parameters>$(find health_bot_description)/config/healthbot_controllers.yaml</parameters>
-   </plugin>
+   </plugin>  -->
    <plugin filename="gz-sim-imu-system" name="gz::sim::systems::Imu"/>
    <plugin filename="gz-sim-sensors-system" name="gz::sim::systems::Sensors">

File: src/health_bot_description/urdf/healthbot_ros2_control.xacro (robot description, xacro)
@@ -1,47 +1,37 @@
 <?xml version="1.0"?>
-<robot xmlns:xacro="http://www.ros.org/wiki/xacro" name="bumperbot">
-    <ros2_control name="RobotSystem" type="system">
-        <!-- ros2_control Gazebo -->
-        <!-- <xacro:if value="$(arg is_sim)"> -->
-            <!-- ROS 2 Humble -->
-            <!-- <xacro:if value="$(arg is_ignition)">
-                <hardware>
-                    <plugin>ign_ros2_control/IgnitionSystem</plugin>
-                </hardware>
-            </xacro:if> -->
-            <!-- ROS 2 Iron or above -->
-            <!-- <xacro:unless value="$(arg is_ignition)">
-                <hardware>
-                    <plugin>gz_ros2_control/GazeboSimSystem</plugin>
-                </hardware>
-            </xacro:unless>
-        </xacro:if> -->
-        <!-- ros2_control Real Robot -->
-        <!-- <xacro:unless value="$(arg is_sim)">
-            <hardware>
-                <plugin>bumperbot_firmware/BumperbotInterface</plugin>
-                <param name="port">/dev/arduino</param>
-            </hardware>
-        </xacro:unless> -->
-        <!-- ros2_control Common Interfaces -->
-        <hardware>
+<robot xmlns:xacro="http://www.ros.org/wiki/xacro" name="healthbot">
+  <ros2_control name="RobotSystem" type="system">
+    <!-- ros2_control Gazebo (Simulation only) -->
+    <xacro:if value="$(arg is_sim)">
+      <hardware>
         <plugin>gz_ros2_control/GazeboSimSystem</plugin>
-        </hardware>
-        <joint name="wheel_right_joint">
-            <command_interface name="velocity">
-              <param name="min">-1</param>
-              <param name="max">1</param>
-            </command_interface>
-            <state_interface name="position" />
-            <state_interface name="velocity" />
-        </joint>
-        <joint name="wheel_left_joint">
-            <command_interface name="velocity">
-              <param name="min">-1</param>
-              <param name="max">1</param>
-            </command_interface>
-            <state_interface name="position" />
-            <state_interface name="velocity" />
-        </joint>
-    </ros2_control>
+      </hardware>
+    </xacro:if>
+    <!-- ros2_control Real Robot (optional, uncomment if you have firmware) -->
+    <!--
+    <xacro:unless value="$(arg is_sim)">
+      <hardware>
+        <plugin>healthbot_firmware/HealthbotInterface</plugin>
+        <param name="port">/dev/arduino</param>
+      </hardware>
+    </xacro:unless>
+    -->
+    <!-- ros2_control Common Interfaces -->
+    <joint name="wheel_right_joint">
+      <command_interface name="velocity">
+        <param name="min">-1</param>
+        <param name="max">1</param>
+      </command_interface>
+      <state_interface name="position"/>
+      <state_interface name="velocity"/>
+    </joint>
+    <joint name="wheel_left_joint">
+      <command_interface name="velocity">
+        <param name="min">-1</param>
+        <param name="max">1</param>
+      </command_interface>
+      <state_interface name="position"/>
+      <state_interface name="velocity"/>
+    </joint>
+  </ros2_control>
 </robot>
