Commit message: robot name changed

File: src/healthrobot_description/urdf/healthrobot.urdf.xacro (robot description, xacro)
@@ -1,4 +1,4 @@
 <?xml version="1.0"?>
-<robot name="health_bot" xmlns:xacro="http://ros.org/wiki/xacro">
+<robot name="healthrobot" xmlns:xacro="http://ros.org/wiki/xacro">
   <!-- Start GZ or Ignition depending on ROS 2 Version -->
   <xacro:arg name="is_ignition" default="true"/>
@@ -6,8 +6,8 @@
   <xacro:arg name="is_sim" default="true"/>
   <!-- Include Gazebo Parameters -->
-  <xacro:include filename="$(find health_bot_description)/urdf/healthbot_gazebo.xacro" />
+  <xacro:include filename="$(find healthrobot_description)/urdf/healthrobot_gazebo.xacro" />
 <!--
   Include ros2_control Plugins -->
-  <xacro:include filename="$(find health_bot_description)/urdf/healthbot_ros2_control.xacro" />
+  <xacro:include filename="$(find healthrobot_description)/urdf/healthrobot_ros2_control.xacro" />
   <link name="base_footprint"/>
   <link name="base_link">
@@ -22,5 +22,5 @@
       <origin xyz="0 0 0" rpy="0 0 0" />
       <geometry>
-        <mesh filename="package://health_bot_description/meshes/base_link.STL" />
+        <mesh filename="package://healthrobot_description/meshes/base_link.STL" />
       </geometry>
       <material name="black"/>
@@ -29,5 +29,5 @@
       <origin xyz="0 0 0" rpy="0 0 0" />
       <geometry>
-        <mesh filename="package://health_bot_description/meshes/base_link.STL" />
+        <mesh filename="package://healthrobot_description/meshes/base_link.STL" />
       </geometry>
     </collision>
@@ -49,5 +49,5 @@
       <origin xyz="0 0 0" rpy="1.57 0 0" />
       <geometry>
-        <mesh filename="package://health_bot_description/meshes/wheel_right_link.STL" />
+        <mesh filename="package://healthrobot_description/meshes/wheel_right_link.STL" />
       </geometry>
       <material name="blue"/>
@@ -78,5 +78,5 @@
       <origin xyz="0 0 0" rpy="-1.57 0 0" />
       <geometry>
-        <mesh filename="package://health_bot_description/meshes/wheel_left_link.STL" />
+        <mesh filename="package://healthrobot_description/meshes/wheel_left_link.STL" />
       </geometry>
       <material name="blue"/>
@@ -106,5 +106,5 @@
       <origin xyz="0 0 0" rpy="0 0 0" />
       <geometry>
-        <mesh filename="package://health_bot_description/meshes/caster_front_link.STL" />
+        <mesh filename="package://healthrobot_description/meshes/caster_front_link.STL" />
       </geometry>
       <material name="silver"/>
@@ -134,5 +134,5 @@
       <origin xyz="0 0 0" rpy="0 0 0" />
       <geometry>
-        <mesh filename="package://health_bot_description/meshes/caster_rear_link.STL" />
+        <mesh filename="package://healthrobot_description/meshes/caster_rear_link.STL" />
       </geometry>
       <material name="silver"/>
@@ -162,5 +162,5 @@
       <origin xyz="0 0 0" rpy="0 0 0" />
       <geometry>
-        <mesh filename="package://health_bot_description/meshes/imu_link.STL" />
+        <mesh filename="package://healthrobot_description/meshes/imu_link.STL" />
       </geometry>
       <material name="blue"/>
@@ -169,5 +169,5 @@
       <origin xyz="0 0 0" rpy="0 0 0" />
       <geometry>
-        <mesh filename="package://health_bot_description/meshes/imu_link.STL" />
+        <mesh filename="package://healthrobot_description/meshes/imu_link.STL" />
       </geometry>
     </collision>
@@ -190,5 +190,5 @@
       <origin xyz="0 0 0" rpy="0 0 0" />
       <geometry>
-        <mesh filename="package://health_bot_description/meshes/laser_link.STL" />
+        <mesh filename="package://healthrobot_description/meshes/laser_link.STL" />
       </geometry>
       <material name="dark_grey"/>
@@ -197,5 +197,5 @@
       <origin xyz="0 0 0" rpy="0 0 0" />
       <geometry>
-        <mesh filename="package://health_bot_description/meshes/laser_link.STL" />
+        <mesh filename="package://healthrobot_description/meshes/laser_link.STL" />
       </geometry>
     </collision>

File: src/healthrobot_description/urdf/healthrobot_gazebo.xacro (robot description, xacro)
@@ -42,5 +42,5 @@
   <gazebo>
   <plugin filename="gz_ros2_control-system" name="gz_ros2_control::GazeboSimROS2ControlPlugin" >
-    <parameters>$(find healthbot_ros2_control)/config/healthrobot_controllers.yaml</parameters>
+    <parameters>$(find healthrobot_ros2_control)/config/healthrobot_controllers.yaml</parameters>
   </plugin>
    <plugin filename="gz-sim-imu-system" name="gz::sim::systems::Imu"/>

File: src/healthrobot_description/urdf/healthrobot_ros2_control.xacro (robot description, xacro)
@@ -1,5 +1,5 @@
 <?xml version="1.0"?>
 <robot xmlns:xacro="http://www.ros.org/wiki/xacro" name="healthbot">
-  <ros2_control name="HealthbotSystem" type="system">
+  <ros2_control name="HealthrobotSystem" type="system">
     <!-- ros2_control Gazebo (Simulation only) -->
       <hardware>
